File: Headtracker-Hardware-XIAO-nRF52.kicad_pcb (KiCad board)
At the start: 2 copper layers, 47 x 25.4 mm, 29 parts, among them J1 Conn_01x04, SW1 User sw, SW2 RST, U1 Xiao_nRF52840, U2 *MC5883L, U3 MPU-6500

Commit message: Update Headtracker-Hardware-XIAO-nRF52.kicad_pcb, Headtracker-Hardware-XIAO-nRF52.kicad_sch, PJ320A.STEP, and 1 more file
Parts:
- removed C1, C4, C5, C6: 104, Capacitor_SMD:C_0603_1608Metric_Pad1.08x0.95mm_HandSolder
- removed C2: 0.22uF, Capacitor_SMD:C_0603_1608Metric_Pad1.08x0.95mm_HandSolder
- removed C3: 1.7uF, Capacitor_SMD:C_0603_1608Metric_Pad1.08x0.95mm_HandSolder
- removed C7: 10nF, Capacitor_SMD:C_0603_1608Metric_Pad1.08x0.95mm_HandSolder
- removed C8, C9: 0.1uF, Capacitor_SMD:C_0603_1608Metric_Pad1.08x0.95mm_HandSolder
- removed D1: , Headtracker-Hardware-XIAO-nRF52:LED_SK6812MINI_PLCC4_3.5x3.5mm_P1.75mm
- removed J1: Conn_01x04, Headtracker-Hardware-XIAO-nRF52:SWD-4PIN
- removed JP1: , Jumper:SolderJumper-3_P1.3mm_Bridged12_RoundedPad1.0x1.5mm
- removed R1: 4.7K, Resistor_SMD:R_0603_1608Metric_Pad0.98x0.95mm_HandSolder
- removed R2, R3: 10K, Resistor_SMD:R_0603_1608Metric_Pad0.98x0.95mm_HandSolder
- removed U1: Xiao_nRF52840, Headtracker-Hardware-XIAO-nRF52:XIAO-nRF52840-Sense-14P-2.54-21X17.8MM
- removed U2: *MC5883L, Headtracker-Hardware-XIAO-nRF52:HMC5883L_EXTENDED
- removed U3: MPU-6500, Headtracker-Hardware-XIAO-nRF52:MPU-6500
- removed kibuzzard-64772BFC: G***, kibuzzard-64772BFC
- removed kibuzzard-64774591: G***, kibuzzard-64774591
- removed kibuzzard-6477459A: G***, kibuzzard-6477459A
- removed kibuzzard-647745A0: G***, kibuzzard-647745A0
- removed kibuzzard-647745A5: G***, kibuzzard-647745A5
- removed kibuzzard-6483527C: G***, kibuzzard-6483527C
- added H4: Hole, MountingHole:MountingHole_2.2mm_M2_Pad, F.Cu at (137.2, 40.0)
- added REF**: PJ-320A, Headtracker-Hardware-XIAO-nRF52:PJ-320A, F.Cu at (123.8, 40.9)
- added REF**: USB-C-16pin-hight-v2, kien242:USB-C-16pin-hight-v2, F.Cu at (120.0, 50.8)
- added REF**: JST_SH_SM02B-SRSS-TB_1x02-1MP, kien242:JST_SH_SM02B-SRSS-TB_1x02-1MP, F.Cu at (123.8, 60.3)
- added U5: E73-2G4M08S1C-52840, kien242:E73-2G4M08S1C, F.Cu at (145.8, 50.8)
- added kibuzzard-6496724A: G***, kibuzzard-6496724A, F.Cu at (147.3, 38.1)
- added kibuzzard-6496725B: G***, kibuzzard-6496725B, F.Cu at (147.3, 63.5)
- moved H1 73.5 mm to (157.5, 40.0)
- moved H2 73.5 mm to (157.5, 61.6)
- moved H3 67.4 mm to (137.2, 61.6)
- moved SW1 58.3 mm to (147.3, 61.0), turned to 0 degrees
- moved SW2 58.3 mm to (147.3, 40.6), turned to 0 degrees
Routing:
- net +3.3V: track 52.1 -> 0.00 mm, vias 2 -> 0
- net GND: track 7.10 -> 0.00 mm, vias 2 -> 0
- net SDA: track 4.16 -> 0.00 mm
- net Net-(U3-AD0/SDO): track 3.88 -> 0.00 mm
- net Net-(JP1-C): track 3.27 -> 0.00 mm
- net SCL: track 2.80 -> 0.00 mm
- net Net-(U2-SETC): track 2.67 -> 0.00 mm
- net Net-(U2-C1): track 2.44 -> 0.00 mm
- net Net-(U3-REGOUT): track 2.02 -> 0.00 mm
- net SWDIO: vias 1 -> 0
- net SWCLK: vias 1 -> 0
Other:
- board size 47 x 25.4 mm -> 46.2 x 27.9 mm
